Commit message: Add files via upload

File: arm/xacro/arm.xacro (robot description, xacro)
@@ -431,4 +431,6 @@
 <xacro:macro name="arm">
     <!--bases-->
+    <base_footprint/>
+    <fixed_parent_to_child parent="base_footprint" child="base_pad" x="0" y="0" z="0" fg="0" fy="0" ph="0" />
     <base_pad/>
     <base_joint/>
@@ -474,5 +476,3 @@
     </gazebo>
     </xacro:macro>
-    <!--Main-->
-    <arm/>
 </robot>

File: zzbot/zzbot_description/zzbot.xacro (robot description, xacro)
@@ -9,7 +9,7 @@
 	<zzbot_body/>
 	<!--sensors-->
+	<rplidar/>
 	<imu />
 	<kinect_camera/>
-	<rplidar/>
 	<!--arm-->
 	<fixed_parent_to_child parent="third_link" child="laser_link" x="0" y="0" z="0.025" fg="0" fy="0" ph="0" />
@@ -21,4 +21,5 @@
   	</plugin>
   	</gazebo>
-    <![CDATA[]]>
+    <![CDATA[
+	]]>
 </robot>

File: zzbot/zzbot_description/zzbot_body/zzbot_body.xacro (robot description, xacro)
@@ -360,5 +360,5 @@
                     <cylinder length="${base_length}" radius="${base_radius}"/>
                 </geometry>
-                <material name="yellow" />
+                <material name="Blue" />
             </visual>
             <collision>
@@ -381,5 +381,5 @@
                     <cylinder length="${base_length}" radius="${base_radius}"/>
                 </geometry>
-                <material name="yellow" />
+                <material name="Blue" />
             </visual>
             <collision>
@@ -422,5 +422,5 @@
         <!--left_driver-->
         <motor dir="left" r="1.5707" p="0" y="0" />
-	    <fixed_parent_to_child parent="base_link" child="left_motor" x="${-base_radius/2}" y="${base_radius/2}" z="0" fg="0" fy="0" ph="0"/>
+	    <fixed_parent_to_child parent="base_link" child="left_motor" x="0" y="${base_radius/2}" z="0" fg="0" fy="0" ph="0"/>
         <wheel dir="left" r="1.5707" p="0" y="0" />
         <continuous_parent_to_child parent="left_motor" child="left_wheel" x="0" y="${motor_length/2}" z="0" fg="0" fy="0" ph="0" ax="0" ay="1" az="0" />
@@ -431,5 +431,5 @@
         <!--right_driver-->
         <motor dir="right" r="-1.5707" p="0" y="0" />
-	    <fixed_parent_to_child parent="base_link" child="right_motor" x="${-base_radius/2}" y="${-base_radius/2}" z="0" fg="0" fy="0" ph="0"/>
+	    <fixed_parent_to_child parent="base_link" child="right_motor" x="0" y="${-base_radius/2}" z="0" fg="0" fy="0" ph="0"/>
         <wheel dir="right" r="-1.5707" p="0" y="0" />
         <continuous_parent_to_child parent="right_motor" child="right_wheel" x="0" y="${-motor_length/2}" z="0" fg="0" fy="0" ph="0" ax="0" ay="1" az="0" />
@@ -440,4 +440,5 @@
         <!--front_wheel-->
 	    <front_uni_wheel />
+        <back_uni_wheel />
         <gazebo>
             <plugin name="differential_drive_controller" filename="libgazebo_ros_diff_drive.so">
